File: eagle/MIX0401/MIX0401_Main.brd (EAGLE design)
At the start: 70.8 x 45.7 mm, 30 parts, among them IC1 NJM4580, IC2 NJM4580

Commit message: Update: Eagle files
Parts:
- added R6: 2.2k, rcl:0207/7
- moved C11 12.0 mm to (25.4, 34.3), turned to 90 degrees
- moved R8 8.03 mm to (54.6, 35.6)
- moved C1 7.62 mm to (11.4, 30.5)
- moved C2 5.08 mm to (11.4, 22.9)
- moved C3 2.54 mm to (11.4, 15.2)
- moved C6 2.54 mm to (43.2, 16.5)
- moved R3 2.54 mm to (19.1, 15.2)
- moved R4 2.54 mm to (19.1, 10.2)
- moved C10 2.54 mm to (61.0, 29.2)
- moved C9 2.54 mm to (62.2, 12.7)
- moved IC1 2.54 mm to (36.8, 19.1)
- moved IC2 2.54 mm to (59.7, 19.1)
- moved JP1 2.54 mm to (57.1, 40.6)
- moved JP2 2.54 mm to (57.1, 12.7)
- moved JP3 2.54 mm to (5.08, 20.3)
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Connections:
- new net N$3: IC1.3, R6.2
- net VCC/2: now also R6.1; no longer IC1.3
Routing:
- net GND: track 0.00 -> 238.5 mm, vias 0 -> 4
- net VCC/2: track 0.00 -> 78.7 mm, vias 0 -> 4
- net VCC: track 0.00 -> 76.4 mm
- net N$1: track 0.00 -> 40.6 mm
- net N$4: track 0.00 -> 23.9 mm
- net N$11: track 0.00 -> 22.9 mm
- net N$6: track 0.00 -> 17.8 mm
- net N$13: track 0.00 -> 16.3 mm
- net N$16: track 0.00 -> 13.8 mm
- net N$10: track 0.00 -> 11.2 mm
- net N$15: track 0.00 -> 8.67 mm
- net N$12: track 0.00 -> 7.62 mm
- net N$2: track 0.00 -> 7.18 mm
- net N$5: track 0.00 -> 6.13 mm
- net N$3: track 0.00 -> 5.08 mm
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Other:
- board size 70.8 x 45.7 mm -> 71.2 x 45.7 mm
- board text added: "MIX0401"
- board text added: "http://dad8893.blogspot.jp/"

Commit message: はんだ付け完了
Parts:
- added C12: 47uF, rcl:E2,5-6
- added R12: 100, rcl:0207/7
- R10, R9: value 10k -> 100k
- moved C10 4.02 mm to (62.2, 33.0), turned to 180 degrees
- moved R8 2.54 mm to (54.6, 38.1)
Connections:
- new net N$19: C10.+, R12.1
- net N$12: now also R12.2; no longer C10.+
- net VCC: now also C12.+
- net VCC/2: now also C12.-
Routing:
- net N$19: track 0.00 -> 8.67 mm
- net VCC: track 76.4 -> 84.4 mm
- net VCC/2: track 78.7 -> 84.9 mm
- net N$12: track 7.62 -> 5.08 mm
- net N$10: track 11.2 -> 8.67 mm
- net GND: track 238.5 -> 236.0 mm
Changed lines of the file:
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@@
 <attribute name="SPICEPREFIX" value="C" x="11.43" y="30.48" size="1.778" layer="27" rot="R180" display="off"/>
 </element>
-<element name="C10" library="rcl" library_urn="urn:adsk.eagle:library:334" package="E2,5-7" package3d_urn="urn:adsk.eagle:package:23345/1" value="100uF" x="60.96" y="29.21" rot="R90">
-<attribute name="SPICEPREFIX" value="C" x="60.96" y="29.21" size="1.778" layer="27" rot="R90" display="off"/>
-</element>
-<element name="C11" library="rcl" library_urn="urn:adsk.eagle:library:334" package="E2,5-7" package3d_urn="urn:adsk.eagle:package:23345/1" value="100uF" x="25.4" y="34.29" rot="R90">
+<element name="C10" library="rcl" library_urn="urn:adsk.eagle:library:334" package="E2,5-7" package3d_urn="urn:adsk.eagle:package:23345/1" value="100uF" x="62.23" y="33.02" rot="R180">
+<attribute name="SPICEPREFIX" value="C" x="62.23" y="33.02" size="1.778" layer="27" rot="R180" display="off"/>
+</element>
+<element name="C11" library="rcl" library_urn="urn:adsk.eagle:library:334" package="E2,5-7" package3d_urn="urn:adsk.eagle:package:23345/1" value="100uF" x="25.4" y="34.29" smashed="yes" rot="R90">
+<attribute name="NAME" x="23.622" y="30.988" size="1.27" layer="25" ratio="10" rot="R180"/>
 <attribute name="SPICEPREFIX" value="C" x="25.4" y="34.29" size="1.778" layer="27" rot="R90" display="off"/>
+<attribute name="VALUE" x="28.575" y="37.338" size="1.27" layer="27" ratio="10" rot="R90"/>
 </element>
 <element name="C13" library="rcl" library_urn="urn:adsk.eagle:library:334" package="E2,5-6" package3d_urn="urn:adsk.eagle:package:23349/1" value="47uF" x="40.64" y="26.67" rot="R90">
@@
 <attribute name="SPICEPREFIX" value="R" x="19.05" y="25.4" size="1.778" layer="27" display="off"/>
 </element>
-<element name="R10" library="rcl" library_urn="urn:adsk.eagle:library:334" package="0207/7" package3d_urn="urn:adsk.eagle:package:23493/1" value="10k" x="35.56" y="29.21" smashed="yes" rot="R90">
+<element name="R10" library="rcl" library_urn="urn:adsk.eagle:library:334" package="0207/7" package3d_urn="urn:adsk.eagle:package:23493/1" value="100k" x="35.56" y="29.21" smashed="yes" rot="R90">
 <attribute name="NAME" x="36.703" y="34.29" size="1.27" layer="25" ratio="10" rot="R90"/>
 <attribute name="SPICEPREFIX" value="R" x="35.56" y="29.21" size="1.778" layer="27" rot="R90" display="off"/>
@@
 <attribute name="VALUE" x="34.544" y="12.1412" size="1.27" layer="27" ratio="10"/>
 </element>
-<element name="R8" library="rcl" library_urn="urn:adsk.eagle:library:334" package="0207/7" package3d_urn="urn:adsk.eagle:package:23493/1" value="100k" x="54.61" y="35.56">
-<attribute name="SPICEPREFIX" value="R" x="54.61" y="35.56" size="1.778" layer="27" display="off"/>
-</element>
-<element name="R9" library="rcl" library_urn="urn:adsk.eagle:library:334" package="0207/7" package3d_urn="urn:adsk.eagle:package:23493/1" value="10k" x="33.02" y="29.21" smashed="yes" rot="R270">
+<element name="R8" library="rcl" library_urn="urn:adsk.eagle:library:334" package="0207/7" package3d_urn="urn:adsk.eagle:package:23493/1" value="100k" x="54.61" y="38.1">
+<attribute name="SPICEPREFIX" value="R" x="54.61" y="38.1" size="1.778" layer="27" display="off"/>
+</element>
+<element name="R9" library="rcl" library_urn="urn:adsk.eagle:library:334" package="0207/7" package3d_urn="urn:adsk.eagle:package:23493/1" value="100k" x="33.02" y="29.21" smashed="yes" rot="R270">
 <attribute name="NAME" x="33.147" y="36.83" size="1.27" layer="25" ratio="10" rot="R270"/>
 <attribute name="SPICEPREFIX" value="R" x="33.02" y="29.21" size="1.778" layer="27" rot="R270" display="off"/>
@@
 <attribute name="SPICEPREFIX" value="R" x="34.29" y="10.16" size="1.778" layer="27" display="off"/>
 <attribute name="VALUE" x="32.004" y="9.6012" size="1.27" layer="27" ratio="10"/>
+</element>
+<element name="R12" library="rcl" library_urn="urn:adsk.eagle:library:334" package="0207/7" package3d_urn="urn:adsk.eagle:package:23493/1" value="100" x="62.23" y="25.4" smashed="yes" rot="R180">
+<attribute name="NAME" x="62.23" y="27.813" size="1.27" layer="25" ratio="10" rot="R180"/>
+<attribute name="SPICEPREFIX" value="R" x="62.23" y="25.4" size="1.778" layer="27" rot="R180" display="off"/>
+<attribute name="VALUE" x="64.516" y="25.9588" size="1.27" layer="27" ratio="10" rot="R180"/>
+</element>
+<element name="C12" library="rcl" library_urn="urn:adsk.eagle:library:334" package="E2,5-6" package3d_urn="urn:adsk.eagle:package:23349/1" value="47uF" x="48.26" y="26.67" rot="R270">
+<attribute name="SPICEPREFIX" value="C" x="48.26" y="26.67" size="1.778" layer="27" rot="R270" display="off"/>
 </element>
 </elements>
@@
 <wire x1="30.48" y1="20.32" x2="35.56" y2="20.32" width="0.4064" layer="16"/>
 <wire x1="35.56" y1="20.32" x2="43.18" y2="20.32" width="0.4064" layer="16"/>
-<wire x1="43.18" y1="20.32" x2="53.34" y2="20.32" width="0.4064" layer="16"/>
+<wire x1="43.18" y1="20.32" x2="45.72" y2="20.32" width="0.4064" layer="16"/>
+<wire x1="45.72" y1="20.32" x2="53.34" y2="20.32" width="0.4064" layer="16"/>
 <wire x1="27.94" y1="20.32" x2="30.48" y2="20.32" width="0.4064" layer="16"/>
 <wire x1="30.48" y1="10.16" x2="27.94" y2="10.16" width="0.4064" layer="16"/>
@@
 <via x="53.34" y="12.7" extent="1-16" drill="0.35"/>
 <via x="53.34" y="7.62" extent="1-16" drill="0.35"/>
+<contactref element="C12" pad="-"/>
+<wire x1="48.26" y1="25.4" x2="45.72" y2="22.86" width="0.4064" layer="16"/>
+<wire x1="45.72" y1="22.86" x2="45.72" y2="20.32" width="0.4064" layer="16"/>
 </signal>
 <signal name="VCC">
@@
 <wire x1="15.24" y1="35.56" x2="17.78" y2="33.02" width="0.4064" layer="16"/>
 <wire x1="17.78" y1="33.02" x2="25.4" y2="33.02" width="0.4064" layer="16"/>
-<wire x1="30.48" y1="35.56" x2="45.72" y2="35.56" width="0.4064" layer="16"/>
+<wire x1="30.48" y1="35.56" x2="50.8" y2="35.56" width="0.4064" layer="16"/>
 <wire x1="33.02" y1="25.4" x2="25.4" y2="25.4" width="0.4064" layer="16"/>
 <wire x1="25.4" y1="25.4" x2="25.4" y2="33.02" width="0.4064" layer="16"/>
 <wire x1="25.4" y1="33.02" x2="27.94" y2="33.02" width="0.4064" layer="16"/>
 <wire x1="27.94" y1="33.02" x2="30.48" y2="35.56" width="0.4064" layer="16"/>
+<wire x1="53.34" y1="33.02" x2="53.34" y2="27.94" width="0.4064" layer="16"/>
 <wire x1="53.34" y1="27.94" x2="53.34" y2="22.86" width="0.4064" layer="16"/>
-<wire x1="45.72" y1="35.56" x2="53.34" y2="27.94" width="0.4064" layer="16"/>
+<wire x1="50.8" y1="35.56" x2="53.34" y2="33.02" width="0.4064" layer="16"/>
 <wire x1="53.34" y1="22.86" x2="55.88" y2="22.86" width="0.4064" layer="16"/>
+<contactref element="C12" pad="+"/>
+<wire x1="48.26" y1="27.94" x2="53.34" y2="27.94" width="0.4064" layer="16"/>
 </signal>
 <signal name="GND">
@@
 <wire x1="40.64" y1="43.18" x2="50.8" y2="43.18" width="1.016" layer="16"/>
 <wire x1="55.88" y1="40.64" x2="55.88" y2="30.48" width="1.016" layer="16"/>
-<wire x1="50.8" y1="35.56" x2="50.8" y2="43.18" width="1.016" layer="16"/>
+<wire x1="50.8" y1="38.1" x2="50.8" y2="43.18" width="1.016" layer="16"/>
 <wire x1="55.88" y1="43.18" x2="50.8" y2="43.18" width="1.016" layer="16"/>
 <wire x1="55.88" y1="40.64" x2="55.88" y2="43.18" width="1.016" layer="16"/>
@@
 <contactref element="IC2" pad="6"/>
 <contactref element="IC2" pad="7"/>
-<contactref element="C10" pad="+"/>
 <wire x1="58.42" y1="22.86" x2="60.96" y2="22.86" width="0.4064" layer="16"/>
-<wire x1="60.96" y1="22.86" x2="60.96" y2="27.94" width="0.4064" layer="16"/>
+<contactref element="R12" pad="2"/>
+<wire x1="58.42" y1="22.86" x2="58.42" y2="25.4" width="0.4064" layer="16"/>
 </signal>
 <signal name="N$13">
@@
 </signal>
 <signal name="N$10">
-<contactref element="JP1" pad="1"/>
 <contactref element="R8" pad="2"/>
 <contactref element="C10" pad="-"/>
-<wire x1="58.42" y1="40.64" x2="58.42" y2="35.56" width="0.4064" layer="16"/>
-<wire x1="58.42" y1="35.56" x2="60.96" y2="33.02" width="0.4064" layer="16"/>
-<wire x1="60.96" y1="33.02" x2="60.96" y2="30.48" width="0.4064" layer="16"/>
+<contactref element="JP1" pad="1"/>
+<wire x1="58.42" y1="40.64" x2="58.42" y2="38.1" width="0.4064" layer="16"/>
+<wire x1="60.96" y1="33.02" x2="60.96" y2="35.56" width="0.4064" layer="16"/>
+<wire x1="60.96" y1="35.56" x2="58.42" y2="38.1" width="0.4064" layer="16"/>
 </signal>
 <signal name="N$11">
@@
 <wire x1="38.1" y1="15.24" x2="38.1" y2="10.16" width="0.4064" layer="16"/>
 </signal>
+<signal name="N$19">
+<contactref element="R12" pad="1"/>
+<contactref element="C10" pad="+"/>
+<wire x1="66.04" y1="25.4" x2="66.04" y2="30.48" width="0.4064" layer="16"/>
+<wire x1="66.04" y1="30.48" x2="63.5" y2="33.02" width="0.4064" layer="16"/>
+</signal>
 </signals>
