File: eagle/MIX0401/MIX0401_Main.sch (EAGLE design)
At the start: 30 parts, among them IC1 NJM4580, IC2 NJM4580

Commit message: Update: Eagle files
Parts:
- added R6: 2.2k, rcl:R-EU_0207/7
Connections:
- new net N$3: IC1A.+IN, R6.2
- net VCC/2: now also R6.1; no longer IC1A.+IN
Other:
- moved on the sheet: C1, C10, C11, C13, C2, C3, C4, C5, C6, C7, C8, C9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

Commit message: はんだ付け完了
Parts:
- added C12: 47uF, rcl:CPOL-EUE2.5-6
- added R12: 100, rcl:R-EU_0207/7
- R10, R9: value 10k -> 100k
Connections:
- new net N$19: C10.+, R12.1
- net N$12: now also R12.2; no longer C10.+
- net VCC: now also C12.+
- net VCC/2: now also C12.-
Other:
- moved on the sheet: C10, JP1, R8
Changed lines of the file:
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@@
 <part name="GND5" library="supply1" library_urn="urn:adsk.eagle:library:371" deviceset="GND" device=""/>
 <part name="GND6" library="supply1" library_urn="urn:adsk.eagle:library:371" deviceset="GND" device=""/>
-<part name="R9" library="rcl" library_urn="urn:adsk.eagle:library:334" deviceset="R-EU_" device="0207/7" package3d_urn="urn:adsk.eagle:package:23493/1" value="10k"/>
-<part name="R10" library="rcl" library_urn="urn:adsk.eagle:library:334" deviceset="R-EU_" device="0207/7" package3d_urn="urn:adsk.eagle:package:23493/1" value="10k"/>
+<part name="R9" library="rcl" library_urn="urn:adsk.eagle:library:334" deviceset="R-EU_" device="0207/7" package3d_urn="urn:adsk.eagle:package:23493/1" value="100k"/>
+<part name="R10" library="rcl" library_urn="urn:adsk.eagle:library:334" deviceset="R-EU_" device="0207/7" package3d_urn="urn:adsk.eagle:package:23493/1" value="100k"/>
 <part name="P+7" library="supply1" library_urn="urn:adsk.eagle:library:371" deviceset="VCC" device=""/>
 <part name="GND7" library="supply1" library_urn="urn:adsk.eagle:library:371" deviceset="GND" device=""/>
@@
 <part name="R6" library="rcl" library_urn="urn:adsk.eagle:library:334" deviceset="R-EU_" device="0207/7" package3d_urn="urn:adsk.eagle:package:23493/1" value="2.2k"/>
 <part name="FRAME1" library="frames" library_urn="urn:adsk.eagle:library:229" deviceset="A4L-LOC" device="" value="Frame"/>
+<part name="R12" library="rcl" library_urn="urn:adsk.eagle:library:334" deviceset="R-EU_" device="0207/7" package3d_urn="urn:adsk.eagle:package:23493/1" value="100"/>
+<part name="C12" library="rcl" library_urn="urn:adsk.eagle:library:334" deviceset="CPOL-EU" device="E2.5-6" package3d_urn="urn:adsk.eagle:package:23349/1" value="47uF"/>
 </parts>
 <sheets>
@@
 <plain>
 <text x="38.1" y="157.48" size="2.54" layer="91">PWR</text>
-<text x="190.5" y="83.82" size="2.54" layer="91">Buffer</text>
+<text x="203.2" y="83.82" size="2.54" layer="91">Buffer</text>
 <text x="68.58" y="83.82" size="2.54" layer="91">Summing</text>
 <text x="157.48" y="88.9" size="2.54" layer="91">Amp</text>
@@
 <instance part="GND1" gate="1" x="99.06" y="53.34"/>
 <instance part="C7" gate="G$1" x="101.6" y="101.6" rot="R90"/>
-<instance part="JP1" gate="G$1" x="218.44" y="71.12"/>
+<instance part="JP1" gate="G$1" x="231.14" y="71.12"/>
 <instance part="JP2" gate="G$1" x="147.32" y="88.9" smashed="yes" rot="R90">
 <attribute name="NAME" x="141.605" y="82.55" size="1.778" layer="95" rot="R90"/>
@@
 <instance part="GND4" gate="1" x="177.8" y="50.8"/>
 <instance part="C9" gate="G$1" x="182.88" y="58.42" rot="MR270"/>
-<instance part="R8" gate="G$1" x="200.66" y="63.5" rot="R90"/>
-<instance part="GND5" gate="1" x="200.66" y="53.34"/>
-<instance part="GND6" gate="1" x="208.28" y="53.34"/>
+<instance part="R8" gate="G$1" x="213.36" y="63.5" rot="R90"/>
+<instance part="GND5" gate="1" x="213.36" y="53.34"/>
+<instance part="GND6" gate="1" x="220.98" y="53.34"/>
 <instance part="R9" gate="G$1" x="88.9" y="139.7" rot="R90"/>
 <instance part="R10" gate="G$1" x="88.9" y="124.46" rot="R90"/>
@@
 <instance part="C3" gate="G$1" x="60.96" y="60.96" rot="R270"/>
 <instance part="C4" gate="G$1" x="60.96" y="53.34" rot="R270"/>
-<instance part="C10" gate="G$1" x="193.04" y="73.66" rot="R90"/>
+<instance part="C10" gate="G$1" x="205.74" y="73.66" rot="R90"/>
 <instance part="C11" gate="G$1" x="53.34" y="134.62"/>
 <instance part="C13" gate="G$1" x="121.92" y="127"/>
@@
 <instance part="R6" gate="G$1" x="88.9" y="63.5" rot="R90"/>
 <instance part="FRAME1" gate="G$1" x="0" y="0"/>
+<instance part="R12" gate="G$1" x="195.58" y="73.66" rot="R180"/>
+<instance part="C12" gate="G$1" x="121.92" y="142.24"/>
 </instances>
 <busses>
@@
 <junction x="116.84" y="134.62"/>
 <label x="129.54" y="134.62" size="1.778" layer="95"/>
+<pinref part="C12" gate="G$1" pin="-"/>
+<wire x1="121.92" y1="137.16" x2="121.92" y2="134.62" width="0.1524" layer="91"/>
 </segment>
 <segment>
@@
 <junction x="78.74" y="147.32"/>
 <junction x="88.9" y="147.32"/>
+<wire x1="88.9" y1="147.32" x2="121.92" y2="147.32" width="0.1524" layer="91"/>
+<pinref part="C12" gate="G$1" pin="+"/>
+<wire x1="121.92" y1="147.32" x2="121.92" y2="144.78" width="0.1524" layer="91"/>
 </segment>
 </net>
@@
 <segment>
 <pinref part="GND6" gate="1" pin="GND"/>
-<wire x1="208.28" y1="55.88" x2="208.28" y2="71.12" width="0.1524" layer="91"/>
+<wire x1="220.98" y1="55.88" x2="220.98" y2="71.12" width="0.1524" layer="91"/>
 <pinref part="JP1" gate="G$1" pin="2"/>
-<wire x1="208.28" y1="71.12" x2="215.9" y2="71.12" width="0.1524" layer="91"/>
+<wire x1="220.98" y1="71.12" x2="228.6" y2="71.12" width="0.1524" layer="91"/>
 </segment>
 <segment>
 <pinref part="GND5" gate="1" pin="GND"/>
 <pinref part="R8" gate="G$1" pin="1"/>
-<wire x1="200.66" y1="55.88" x2="200.66" y2="58.42" width="0.1524" layer="91"/>
+<wire x1="213.36" y1="55.88" x2="213.36" y2="58.42" width="0.1524" layer="91"/>
 </segment>
 <segment>
@@
 <pinref part="IC2" gate="B" pin="OUT"/>
 <wire x1="187.96" y1="73.66" x2="185.42" y2="73.66" width="0.1524" layer="91"/>
+<pinref part="R12" gate="G$1" pin="2"/>
 <wire x1="190.5" y1="73.66" x2="187.96" y2="73.66" width="0.1524" layer="91"/>
 <junction x="187.96" y="73.66"/>
-<pinref part="C10" gate="G$1" pin="+"/>
 </segment>
 </net>
@@
 <net name="N$10" class="0">
 <segment>
+<wire x1="210.82" y1="73.66" x2="213.36" y2="73.66" width="0.1524" layer="91"/>
+<pinref part="R8" gate="G$1" pin="2"/>
+<wire x1="213.36" y1="68.58" x2="213.36" y2="73.66" width="0.1524" layer="91"/>
+<pinref part="C10" gate="G$1" pin="-"/>
 <pinref part="JP1" gate="G$1" pin="1"/>
-<wire x1="198.12" y1="73.66" x2="200.66" y2="73.66" width="0.1524" layer="91"/>
-<pinref part="R8" gate="G$1" pin="2"/>
-<wire x1="200.66" y1="73.66" x2="215.9" y2="73.66" width="0.1524" layer="91"/>
-<wire x1="200.66" y1="68.58" x2="200.66" y2="73.66" width="0.1524" layer="91"/>
-<junction x="200.66" y="73.66"/>
-<pinref part="C10" gate="G$1" pin="-"/>
+<wire x1="228.6" y1="73.66" x2="213.36" y2="73.66" width="0.1524" layer="91"/>
+<junction x="213.36" y="73.66"/>
 </segment>
 </net>
@@
 </segment>
 </net>
+<net name="N$19" class="0">
+<segment>
+<pinref part="R12" gate="G$1" pin="1"/>
+<pinref part="C10" gate="G$1" pin="+"/>
+<wire x1="200.66" y1="73.66" x2="203.2" y2="73.66" width="0.1524" layer="91"/>
+</segment>
+</net>
